Commit message: robot stands and has an IMU now :D

File: ros/src/uvc_robot_description/description/robot.urdf.xacro (robot description, xacro)
@@ -3,3 +3,4 @@
     <xacro:include filename="robot_core.xacro"/>
     <xacro:include filename="ros2_control.xacro"/>
+    <xacro:include filename="imu.xacro"/>
 </robot>

File: ros/src/uvc_robot_description/description/robot_core.xacro (robot description, xacro)
@@ -61,4 +61,5 @@
         <axis xyz="0 0 1"/>
         <limit lower="-10" upper="10" effort="10" velocity="10"/>
+        <dynamics damping="0.5" friction="0.2"/>
     </joint>
     <link name="waist_link">
@@ -90,4 +91,5 @@
         <axis xyz="0 0 1"/>
         <limit lower="-2.356" upper="2.356" effort="1.3729" velocity="7.48"/>
+        <dynamics damping="0.5" friction="0.2"/>
     </joint>
     <link name="head_link">
@@ -119,4 +121,5 @@
         <axis xyz="0 -1 0"/>
         <limit lower="-2.356" upper="2.356" effort="1.3729" velocity="7.48"/>
+        <dynamics damping="0.5" friction="0.2"/>
     </joint>
     <link name="left_shoulder_link">
@@ -147,4 +150,5 @@
         <axis xyz="1 0 0"/>
         <limit lower="-2.356" upper="2.356" effort="1.3729" velocity="7.48"/>
+        <dynamics damping="0.5" friction="0.2"/>
     </joint>
     <link name="left_arm_link">
@@ -201,4 +205,5 @@
         <axis xyz="0 0 1"/>
         <limit lower="-2.356" upper="2.356" effort="1.3729" velocity="7.48"/>
+        <dynamics damping="0.5" friction="0.2"/>
     </joint>
     <link name="left_elbow_link">
@@ -226,4 +231,5 @@
         <axis xyz="0 -1 0"/>
         <limit lower="-2.356" upper="2.356" effort="1.3729" velocity="7.48"/>
+        <dynamics damping="0.5" friction="0.2"/>
     </joint>
     <link name="left_forearm_link">
@@ -278,4 +284,5 @@
         <axis xyz="0 -1 0"/>
         <limit lower="-2.356" upper="2.356" effort="1.3729" velocity="7.48"/>
+        <dynamics damping="0.5" friction="0.2"/>
     </joint>
     <link name="right_shoulder_link">
@@ -306,4 +313,5 @@
         <axis xyz="-1 0 0"/>
         <limit lower="-2.356" upper="2.356" effort="1.3729" velocity="7.48"/>
+        <dynamics damping="0.5" friction="0.2"/>
     </joint>
     <link name="right_arm_link">
@@ -360,4 +368,5 @@
         <axis xyz="0 0 -1"/>
         <limit lower="-2.356" upper="2.356" effort="1.3729" velocity="7.48"/>
+        <dynamics damping="0.5" friction="0.2"/>
     </joint>
     <link name="right_elbow_link">
@@ -385,4 +394,5 @@
         <axis xyz="0 -1 0"/>
         <limit lower="-2.356" upper="2.356" effort="1.3729" velocity="7.48"/>
+        <dynamics damping="0.5" friction="0.2"/>
     </joint>
     <link name="right_forearm_link">
@@ -437,4 +447,5 @@
         <axis xyz="0 0 1"/>
         <limit lower="-2.356" upper="2.356" effort="1.3729" velocity="7.48"/>
+        <dynamics damping="0.5" friction="0.2"/>
     </joint>
     <link name="left_hip1_link">
@@ -462,4 +473,5 @@
         <axis xyz="1 0 0"/>
         <limit lower="-2.356" upper="2.356" effort="1.3729" velocity="7.48"/>
+        <dynamics damping="0.5" friction="0.2"/>
     </joint>
     <link name="left_hip2_link">
@@ -500,4 +512,5 @@
         <origin xyz="-0.0008 0.0113 -0.0387"/>
         <limit lower="-2.356" upper="2.356" effort="1.3729" velocity="7.48"/>
+        <dynamics damping="0.5" friction="0.2"/>
     </joint>
     <link name="left_leg_link">
@@ -551,4 +564,5 @@
         <origin xyz="0.00015 0.0 -0.06375"/>
         <limit lower="-2.356" upper="2.356" effort="1.3729" velocity="7.48"/>
+        <dynamics damping="0.5" friction="0.2"/>
     </joint>
     <link name="left_knee_link">
@@ -602,4 +616,5 @@
         <origin xyz="0.0003 -0.0002 -0.0643"/>
         <limit lower="-2.356" upper="2.356" effort="1.3729" velocity="7.48"/>
+        <dynamics damping="0.5" friction="0.2"/>
     </joint>
     <link name="left_ankle_link">
@@ -640,4 +655,5 @@
         <origin xyz="0 -0.01125 -0.037"/>
         <limit lower="-2.356" upper="2.356" effort="1.3729" velocity="7.48"/>
+        <dynamics damping="0.5" friction="0.2"/>
     </joint>
     <link name="left_foot_link">
@@ -666,4 +682,5 @@
         <axis xyz="0 0 -1"/>
         <limit lower="-2.356" upper="2.356" effort="1.3729" velocity="7.48"/>
+        <dynamics damping="0.5" friction="0.2"/>
     </joint>
     <link name="right_hip1_link">
@@ -691,4 +708,5 @@
         <axis xyz="-1 0 0"/>
         <limit lower="-2.356" upper="2.356" effort="1.3729" velocity="7.48"/>
+        <dynamics damping="0.5" friction="0.2"/>
     </joint>
     <link name="right_hip2_link">
@@ -729,4 +747,5 @@
         <origin xyz="-0.0008 -0.0113 -0.0387"/>
         <limit lower="-2.356" upper="2.356" effort="1.3729" velocity="7.48"/>
+        <dynamics damping="0.5" friction="0.2"/>
     </joint>
     <link name="right_leg_link">
@@ -780,4 +799,5 @@
         <origin xyz="0.00015 0.0 -0.06375"/>
         <limit lower="-2.356" upper="2.356" effort="1.3729" velocity="7.48"/>
+        <dynamics damping="0.5" friction="0.2"/>
     </joint>
     <link name="right_knee_link">
@@ -831,4 +851,5 @@
         <origin xyz="0.0003 0.0002 -0.0643"/>
         <limit lower="-2.356" upper="2.356" effort="1.3729" velocity="7.48"/>
+        <dynamics damping="0.5" friction="0.2"/>
     </joint>
     <link name="right_ankle_link">
@@ -869,4 +890,5 @@
         <origin xyz="0 0.01125 -0.037"/>
         <limit lower="-2.356" upper="2.356" effort="1.3729" velocity="7.48"/>
+        <dynamics damping="0.5" friction="0.2"/>
     </joint>
     <link name="right_foot_link">

File: ros/src/uvc_robot_description/description/ros2_control.xacro (robot description, xacro)
@@ -10,4 +10,5 @@
                     <param name="max">10</param>
                 </command_interface>
+                <state_interface name="effort"/>
                 <state_interface name="velocity"/>
                 <state_interface name="position"/>
@@ -18,4 +19,5 @@
                     <param name="max">10</param>
                 </command_interface>
+                <state_interface name="effort"/>
                 <state_interface name="velocity"/>
                 <state_interface name="position"/>
@@ -26,4 +28,5 @@
                     <param name="max">10</param>
                 </command_interface>
+                <state_interface name="effort"/>
                 <state_interface name="velocity"/>
                 <state_interface name="position"/>
@@ -34,4 +37,5 @@
                     <param name="max">10</param>
                 </command_interface>
+                <state_interface name="effort"/>
                 <state_interface name="velocity"/>
                 <state_interface name="position"/>
@@ -42,4 +46,5 @@
                     <param name="max">10</param>
                 </command_interface>
+                <state_interface name="effort"/>
                 <state_interface name="velocity"/>
                 <state_interface name="position"/>
@@ -50,4 +55,5 @@
                     <param name="max">10</param>
                 </command_interface>
+                <state_interface name="effort"/>
                 <state_interface name="velocity"/>
                 <state_interface name="position"/>
@@ -58,4 +64,5 @@
                     <param name="max">10</param>
                 </command_interface>
+                <state_interface name="effort"/>
                 <state_interface name="velocity"/>
                 <state_interface name="position"/>
@@ -66,4 +73,5 @@
                     <param name="max">10</param>
                 </command_interface>
+                <state_interface name="effort"/>
                 <state_interface name="velocity"/>
                 <state_interface name="position"/>
@@ -74,4 +82,5 @@
                     <param name="max">10</param>
                 </command_interface>
+                <state_interface name="effort"/>
                 <state_interface name="velocity"/>
                 <state_interface name="position"/>
@@ -82,7 +91,129 @@
                     <param name="max">10</param>
                 </command_interface>
-                <state_interface name="velocity"/>
-                <state_interface name="position"/>
-            </joint>
+                <state_interface name="effort"/>
+                <state_interface name="velocity"/>
+                <state_interface name="position"/>
+            </joint>
+            <joint name="left_hip1_joint">
+                <command_interface name="effort">
+                    <param name="min">-10</param>
+                    <param name="max">10</param>
+                </command_interface>
+                <state_interface name="effort"/>
+                <state_interface name="velocity"/>
+                <state_interface name="position"/>
+            </joint>
+            <joint name="left_hip2_joint">
+                <command_interface name="effort">
+                    <param name="min">-10</param>
+                    <param name="max">10</param>
+                </command_interface>
+                <state_interface name="effort"/>
+                <state_interface name="velocity"/>
+                <state_interface name="position"/>
+            </joint>
+            <joint name="left_leg_joint">
+                <command_interface name="effort">
+                    <param name="min">-10</param>
+                    <param name="max">10</param>
+                </command_interface>
+                <state_interface name="effort"/>
+                <state_interface name="velocity"/>
+                <state_interface name="position"/>
+            </joint>
+            <joint name="left_knee_joint">
+                <command_interface name="effort">
+                    <param name="min">-10</param>
+                    <param name="max">10</param>
+                </command_interface>
+                <state_interface name="effort"/>
+                <state_interface name="velocity"/>
+                <state_interface name="position"/>
+            </joint>
+            <joint name="left_ankle_joint">
+                <command_interface name="effort">
+                    <param name="min">-10</param>
+                    <param name="max">10</param>
+                </command_interface>
+                <state_interface name="effort"/>
+                <state_interface name="velocity"/>
+                <state_interface name="position"/>
+            </joint>
+            <joint name="left_foot_joint">
+                <command_interface name="effort">
+                    <param name="min">-10</param>
+                    <param name="max">10</param>
+                </command_interface>
+                <state_interface name="effort"/>
+                <state_interface name="velocity"/>
+                <state_interface name="position"/>
+            </joint>
+            <joint name="right_hip1_joint">
+                <command_interface name="effort">
+                    <param name="min">-10</param>
+                    <param name="max">10</param>
+                </command_interface>
+                <state_interface name="effort"/>
+                <state_interface name="velocity"/>
+                <state_interface name="position"/>
+            </joint>
+            <joint name="right_hip2_joint">
+                <command_interface name="effort">
+                    <param name="min">-10</param>
+                    <param name="max">10</param>
+                </command_interface>
+                <state_interface name="effort"/>
+                <state_interface name="velocity"/>
+                <state_interface name="position"/>
+            </joint>
+            <joint name="right_leg_joint">
+                <command_interface name="effort">
+                    <param name="min">-10</param>
+                    <param name="max">10</param>
+                </command_interface>
+                <state_interface name="effort"/>
+                <state_interface name="velocity"/>
+                <state_interface name="position"/>
+            </joint>
+            <joint name="right_knee_joint">
+                <command_interface name="effort">
+                    <param name="min">-10</param>
+                    <param name="max">10</param>
+                </command_interface>
+                <state_interface name="effort"/>
+                <state_interface name="velocity"/>
+                <state_interface name="position"/>
+            </joint>
+            <joint name="right_ankle_joint">
+                <command_interface name="effort">
+                    <param name="min">-10</param>
+                    <param name="max">10</param>
+                </command_interface>
+                <state_interface name="effort"/>
+                <state_interface name="velocity"/>
+                <state_interface name="position"/>
+            </joint>
+            <joint name="right_foot_joint">
+                <command_interface name="effort">
+                    <param name="min">-10</param>
+                    <param name="max">10</param>
+                </command_interface>
+                <state_interface name="effort"/>
+                <state_interface name="velocity"/>
+                <state_interface name="position"/>
+            </joint>
+            <sensor name="imu_sensor">
+                <param name="frame_id">imu_link</param>
+                <state_interface name="orientation.x"/>
+                <state_interface name="orientation.y"/>
+                <state_interface name="orientation.z"/>
+                <state_interface name="orientation.w"/>
+                <state_interface name="angular_velocity.x"/>
+                <state_interface name="angular_velocity.y"/>
+                <state_interface name="angular_velocity.z"/>
+                <state_interface name="linear_acceleration.x"/>
+                <state_interface name="linear_acceleration.y"/>
+                <state_interface name="linear_acceleration.z"/>
+            </sensor>
     </ros2_control>
     <gazebo>
