Commit message: made urdf!

File: ros/src/uvc_robot_description/description/robot_core.xacro (robot description, xacro)
@@ -15,194 +15,557 @@
     </material>
     <link name="base_link"/>
-    <!-- CHASSIS -->
-    <joint name="chassis_joint" type="fixed">
+    <!-- TORSO -->
+    <joint name="torso_joint" type="fixed">
         <parent link="base_link"/>
-        <child link="chassis"/>
-        <origin xyz="-0.144 0 0"/>
-    </joint>
-    <link name="chassis">
-        <visual>
-            <origin xyz="0.144 0 0.038"/>
-            <geometry>
-                <box size="0.096 0.168 0.048"/>
-            </geometry>
-            <material name="white"/>
-        </visual>
-        <visual>
-            <origin xyz="0.144 0.09 0.038"/>
-            <geometry>
-                <box size="0.288 0.012 0.048"/>
-            </geometry>
-            <material name="white"/>
-        </visual>
-        <visual>
-            <origin xyz="0.144 -0.09 0.038"/>
-            <geometry>
-                <box size="0.288 0.012 0.048"/>
-            </geometry>
-            <material name="white"/>
-        </visual>
-        <visual>
-            <origin xyz="0.00125 0.11995 0.038"/>
-            <geometry>
-                <box size="0.0025 0.0479 0.048"/>
-            </geometry>
-            <material name="white"/>
-        </visual>
-        <visual>
-            <origin xyz="0.00125 -0.11995 0.038"/>
-            <geometry>
-                <box size="0.0025 0.0479 0.048"/>
-            </geometry>
-            <material name="white"/>
-        </visual>
-        <visual>
-            <origin xyz="0.28675 0.11995 0.038"/>
-            <geometry>
-                <box size="0.0025 0.0479 0.048"/>
-            </geometry>
-            <material name="white"/>
-        </visual>
-        <visual>
-            <origin xyz="0.28675 -0.11995 0.038"/>
-            <geometry>
-                <box size="0.0025 0.0479 0.048"/>
-            </geometry>
-            <material name="white"/>
-        </visual>
-        <visual>
-            <origin xyz="0.144 0.14515 0.038"/>
-            <geometry>
-                <box size="0.288 0.0025 0.048"/>
-            </geometry>
-            <material name="white"/>
-        </visual>
-        <visual>
-            <origin xyz="0.144 -0.14515 0.038"/>
-            <geometry>
-                <box size="0.288 0.0025 0.048"/>
+        <child link="torso_link"/>
+        <origin xyz="0 0 0.34"/>
+    </joint>
+    <link name="torso_link">
+        <visual>
+            <origin xyz="-0.00475 0 -0.01675"/>
+            <geometry>
+                <box size="0.0805 0.089 0.0605"/>
+            </geometry>
+            <material name="white"/>
+        </visual>
+        <visual>
+            <origin xyz="-0.06925 0 -0.012"/>
+            <geometry>
+                <box size="0.0455 0.105 0.088"/>
+            </geometry>
+            <material name="white"/>
+        </visual>
+    </link>
+    <joint name="waist_joint" type="revolute">
+        <parent link="torso_link"/>
+        <child link="waist_link"/>
+        <origin xyz="-0.02425 0 -0.04715"/>
+        <axis xyz="0 0 1"/>
+        <limit lower="-10" upper="10" effort="10" velocity="10"/>
+    </joint>
+    <link name="waist_link">
+        <visual>
+            <origin xyz="-0.00275 0 -0.022"/>
+            <geometry>
+                <box size="0.0505 0.076 0.036"/>
+            </geometry>
+            <material name="white"/>
+        </visual>
+    </link>
+    <!-- HEAD -->
+    <joint name="head_joint" type="revolute">
+        <parent link="torso_link"/>
+        <child link="head_link"/>
+        <origin xyz="-0.00395 0 0.0134"/>
+        <axis xyz="0 0 1"/>
+        <limit lower="-2.356" upper="2.356" effort="1.3729" velocity="7.48"/>
+    </joint>
+    <link name="head_link">
+        <visual>
+            <origin xyz="0.00225 0 0.0245"/>
+            <geometry>
+                <box size="0.0495 0.032 0.038"/>
             </geometry>
             <material name="white"/>
         </visual>
         <collision>
-            <origin xyz="0.144 0 0.038"/>
-            <geometry>
-                <box size="0.288 0.2928 0.048"/>
+            <origin xyz="0.00225 0 0.0245"/>
+            <geometry>
+                <box size="0.0495 0.032 0.038"/>
             </geometry>
         </collision>
-        <xacro:inertial_box mass="0.5" x="0.288" y="0.2928" z="0.048">
-            <origin xyz="0.144 0 0.038" rpy="0 0 0"/>
+        <xacro:inertial_box mass="0.025" x="0.0495" y="0.032" z="0.038">
+            <origin xyz="0.00225 0 0.0245" rpy="0 0 0"/>
         </xacro:inertial_box>
     </link>
-    <gazebo reference="chassis">
-        <material>Gazebo/White</material>
-    </gazebo>
-    <joint name="front_left_wheel_joint" type="continuous">
-        <parent link="base_link"/>
-        <child link="front_left_wheel"/>
-        <origin xyz="0.096 0.121 0.038" rpy="-${pi/2} 0 0"/>
+    <!-- LEFT ARM -->
+    <joint name="left_shoulder_joint" type="revolute">
+        <parent link="torso_link"/>
+        <child link="left_shoulder_link"/>
+        <origin xyz="-0.0041 0.04725 -0.0009"/>
+        <axis xyz="0 -1 0"/>
+        <limit lower="-2.356" upper="2.356" effort="1.3729" velocity="7.48"/>
+    </joint>
+    <link name="left_shoulder_link">
+        <visual>
+            <origin xyz="0 0.0175 0"/>
+            <geometry>
+                <box size="0.0465 0.036 0.02"/>
+            </geometry>
+            <material name="white"/>
+        </visual>
+        <collision>
+            <origin xyz="0 0.0175 0"/>
+            <geometry>
+                <box size="0.0465 0.036 0.02"/>
+            </geometry>
+        </collision>
+    </link>
+    <joint name="left_arm_joint" type="revolute">
+        <parent link="left_shoulder_link"/>
+        <child link="left_arm_link"/>
+        <origin xyz="0 0.02645 0"/>
+        <axis xyz="1 0 0"/>
+        <limit lower="-2.356" upper="2.356" effort="1.3729" velocity="7.48"/>
+    </joint>
+    <link name="left_arm_link">
+        <visual>
+            <origin xyz=" 0.00025 0 -0.01125"/>
+            <geometry>
+                <box size="0.0355 0.025 0.0425"/>
+            </geometry>
+            <material name="white"/>
+        </visual>
+        <visual>
+            <origin xyz="-0.01175 -0.00025 -0.04825"/>
+            <geometry>
+                <box size="0.0425 0.0225 0.0315"/>
+            </geometry>
+            <material name="white"/>
+        </visual>
+        <visual>
+            <origin xyz="-0.01125 -0.00025 -0.06875"/>
+            <geometry>
+                <box size="0.0505 0.0335 0.0095"/>
+            </geometry>
+            <material name="white"/>
+        </visual>
+    </link>
+    <joint name="left_elbow_joint" type="revolute">
+        <parent link="left_arm_link"/>
+        <child link="left_elbow_link"/>
+        <origin xyz="0.00225 -0.00025 -0.07365"/>
         <axis xyz="0 0 1"/>
-    </joint>
-    <link name="front_left_wheel">
-        <visual>
-            <geometry>
-                <cylinder radius="0.038" length="0.0408"/>
-            </geometry>
-            <material name="blue"/>
+        <limit lower="-2.356" upper="2.356" effort="1.3729" velocity="7.48"/>
+    </joint>
+    <link name="left_elbow_link">
+        <visual>
+            <origin xyz="-0.009 0 -0.012"/>
+            <geometry>
+                <box size="0.042 0.032 0.024"/>
+            </geometry>
+            <material name="white"/>
+        </visual>
+    </link>
+    <joint name="left_forearm_joint" type="revolute">
+        <parent link="left_elbow_link"/>
+        <child link="left_forearm_link"/>
+        <origin xyz="0.0022 0.0 -0.0117"/>
+        <axis xyz="0 -1 0"/>
+        <limit lower="-2.356" upper="2.356" effort="1.3729" velocity="7.48"/>
+    </joint>
+    <link name="left_forearm_link">
+        <visual>
+            <origin xyz="0 0 -0.009"/>
+            <geometry>
+                <box size="0.02 0.0465 0.036"/>
+            </geometry>
+            <material name="white"/>
+        </visual>
+        <visual>
+            <origin xyz="0.001 0 -0.0465"/>
+            <geometry>
+                <box size="0.021 0.032 0.04"/>
+            </geometry>
+            <material name="white"/>
+        </visual>
+        <visual>
+            <origin xyz="0.003 -0.00175 -0.0785"/>
+            <geometry>
+                <box size="0.029 0.0235 0.024"/>
+            </geometry>
+            <material name="white"/>
+        </visual>
+        <visual>
+            <origin xyz="0 0.001 -0.094"/>
+            <geometry>
+                <box size="0.0065 0.0175 0.024" rpy="-0.357409 -0.862853 -0.357411 -1.71778"/>
+            </geometry>
+            <material name="white"/>
+        </visual>
+    </link>
+    <!-- RIGHT ARM -->
+    <joint name="right_shoulder_joint" type="revolute">
+        <parent link="torso_link"/>
+        <child link="right_shoulder_link"/>
+        <origin xyz="-0.0041 -0.04725 -0.0009"/>
+        <axis xyz="0 -1 0"/>
+        <limit lower="-2.356" upper="2.356" effort="1.3729" velocity="7.48"/>
+    </joint>
+    <link name="right_shoulder_link">
+        <visual>
+            <origin xyz="0 -0.0175 0"/>
+            <geometry>
+                <box size="0.0465 0.036 0.02"/>
+            </geometry>
+            <material name="white"/>
         </visual>
         <collision>
-            <geometry>
-                <cylinder radius="0.038" length="0.0408"/>
+            <origin xyz="0 -0.0175 0"/>
+            <geometry>
+                <box size="0.0465 0.036 0.02"/>
             </geometry>
         </collision>
-        <xacro:inertial_cylinder mass="0.1" length="0.038" radius="0.0408">
-            <origin xyz="0 0 0" rpy="0 0 0"/>
-        </xacro:inertial_cylinder>
-    </link>
-    <gazebo reference="front_left_wheel">
-        <material>Gazebo/Blue</material>
-        <mu1 value="0.0"/>
-        <mu2 value="0.0"/>
-    </gazebo>
-    <joint name="back_left_wheel_joint" type="continuous">
-        <parent link="base_link"/>
-        <child link="back_left_wheel"/>
-        <origin xyz="-0.096 0.121 0.038" rpy="-${pi/2} 0 0"/>
+    </link>
+    <joint name="right_arm_joint" type="revolute">
+        <parent link="right_shoulder_link"/>
+        <child link="right_arm_link"/>
+        <origin xyz="0 -0.02645 0"/>
+        <axis xyz="-1 0 0"/>
+        <limit lower="-2.356" upper="2.356" effort="1.3729" velocity="7.48"/>
+    </joint>
+    <link name="right_arm_link">
+        <visual>
+            <origin xyz=" 0.00025 0 -0.01125"/>
+            <geometry>
+                <box size="0.0355 0.025 0.0425"/>
+            </geometry>
+            <material name="white"/>
+        </visual>
+        <visual>
+            <origin xyz="-0.01175 0.00025 -0.04825"/>
+            <geometry>
+                <box size="0.0425 0.0225 0.0315"/>
+            </geometry>
+            <material name="white"/>
+        </visual>
+        <visual>
+            <origin xyz="-0.01125 0.00025 -0.06875"/>
+            <geometry>
+                <box size="0.0505 0.0335 0.0095"/>
+            </geometry>
+            <material name="white"/>
+        </visual>
+    </link>
+    <joint name="right_elbow_joint" type="revolute">
+        <parent link="right_arm_link"/>
+        <child link="right_elbow_link"/>
+        <origin xyz="0.00225 0.00025 -0.07365"/>
+        <axis xyz="0 0 -1"/>
+        <limit lower="-2.356" upper="2.356" effort="1.3729" velocity="7.48"/>
+    </joint>
+    <link name="right_elbow_link">
+        <visual>
+            <origin xyz="-0.009 0 -0.012"/>
+            <geometry>
+                <box size="0.042 0.032 0.024"/>
+            </geometry>
+            <material name="white"/>
+        </visual>
+    </link>
+    <joint name="right_forearm_joint" type="revolute">
+        <parent link="right_elbow_link"/>
+        <child link="right_forearm_link"/>
+        <origin xyz="0.0022 0.0 -0.0117"/>
+        <axis xyz="0 -1 0"/>
+        <limit lower="-2.356" upper="2.356" effort="1.3729" velocity="7.48"/>
+    </joint>
+    <link name="right_forearm_link">
+        <visual>
+            <origin xyz="0 0 -0.009"/>
+            <geometry>
+                <box size="0.02 0.0465 0.036"/>
+            </geometry>
+            <material name="white"/>
+        </visual>
+        <visual>
+            <origin xyz="0.001 0 -0.0465"/>
+            <geometry>
+                <box size="0.021 0.032 0.04"/>
+            </geometry>
+            <material name="white"/>
+        </visual>
+        <visual>
+            <origin xyz="0.003 0.00175 -0.0785"/>
+            <geometry>
+                <box size="0.029 0.0235 0.024"/>
+            </geometry>
+            <material name="white"/>
+        </visual>
+        <visual>
+            <origin xyz="0 -0.001 -0.094"/>
+            <geometry>
+                <box size="0.0065 0.0175 0.024" rpy="-0.357409 -0.862853 -0.357411 -1.71778"/>
+            </geometry>
+            <material name="white"/>
+        </visual>
+    </link>
+    <!-- LEFT LEG -->
+    <joint name="left_hip1_joint" type="revolute">
+        <parent link="waist_link"/>
+        <child link="left_hip1_link"/>
+        <origin xyz="0.00875 0.02145 -0.03995"/>
         <axis xyz="0 0 1"/>
-    </joint>
-    <link name="back_left_wheel">
-        <visual>
-            <geometry>
-                <cylinder radius="0.038" length="0.0408"/>
-            </geometry>
-            <material name="blue"/>
-        </visual>
-        <collision>
-            <geometry>
-                <cylinder radius="0.038" length="0.0408"/>
-            </geometry>
-        </collision>
-        <xacro:inertial_cylinder mass="0.1" length="0.038" radius="0.0408">
-            <origin xyz="0 0 0" rpy="0 0 0"/>
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
Commit message: fixed model rotations

File: ros/src/uvc_robot_description/description/robot_core.xacro (robot description, xacro)
@@ -46,5 +46,5 @@
     <link name="waist_link">
         <visual>
-            <origin xyz="-0.00275 0 -0.022"/>
+            <origin xyz="0.00275 0 -0.022"/>
             <geometry>
                 <box size="0.0505 0.076 0.036"/>
@@ -76,5 +76,5 @@
         </collision>
         <xacro:inertial_box mass="0.025" x="0.0495" y="0.032" z="0.038">
-            <origin xyz="0.00225 0 0.0245" rpy="0 0 0"/>
+            <origin xyz="0.00225 0 0.0245"/>
         </xacro:inertial_box>
     </link>
@@ -177,11 +177,4 @@
             <material name="white"/>
         </visual>
-        <visual>
-            <origin xyz="0 0.001 -0.094"/>
-            <geometry>
-                <box size="0.0065 0.0175 0.024" rpy="-0.357409 -0.862853 -0.357411 -1.71778"/>
-            </geometry>
-            <material name="white"/>
-        </visual>
     </link>
     <!-- RIGHT ARM -->
@@ -283,11 +276,4 @@
             <material name="white"/>
         </visual>
-        <visual>
-            <origin xyz="0 -0.001 -0.094"/>
-            <geometry>
-                <box size="0.0065 0.0175 0.024" rpy="-0.357409 -0.862853 -0.357411 -1.71778"/>
-            </geometry>
-            <material name="white"/>
-        </visual>
     </link>
     <!-- LEFT LEG -->
@@ -347,14 +333,14 @@
         </visual>
         <visual>
-            <origin xyz="0.006 0.0 -0.054"/>
-            <geometry>
-                <box size="0.032 0.042 0.0225" rpy="0.654047 0.654046 0.380062 2.415205"/>
-            </geometry>
-            <material name="white"/>
-        </visual>
-        <visual>
-            <origin xyz="0.003 0 -0.037"/>
-            <geometry>
-                <box size="0.0465 0.036 0.02" rpy="-0.697151 -0.697152 -0.167211 -2.810252"/>
+            <origin xyz="0.006 0.0 -0.054" rpy="2.0887992 -0.0000101 1.5708007"/>
+            <geometry>
+                <box size="0.032 0.042 0.0225"/>
+            </geometry>
+            <material name="white"/>
+        </visual>
+        <visual>
+            <origin xyz="0.003 0 -0.037" rpy="2.6707995 -0.0000107 1.5708003"/>
+            <geometry>
+                <box size="0.0465 0.036 0.02"/>
             </geometry>
             <material name="white"/>
@@ -370,7 +356,7 @@
     <link name="left_knee_link">
         <visual>
-            <origin xyz="0.00425 0 -0.008"/>
-            <geometry>
-                <box size="0.0465 0.036 0.02"  rpy=" 0.454459 0.454452 0.76612 1.834125"/>
+            <origin xyz="0.00425 0 -0.008" rpy="1.0707999 -0.000011 1.5707994"/>
+            <geometry>
+                <box size="0.0465 0.036 0.02"/>
             </geometry>
             <material name="white"/>
@@ -384,7 +370,7 @@
         </visual>
         <visual>
-            <origin xyz="0.004 0.0 -0.054"/>
-            <geometry>
-                <box size="0.032 0.042 0.023"  rpy="-0.63513 -0.635128 -0.43957 -2.313314"/>
+            <origin xyz="0.004 0.0 -0.054" rpy="1.9307994 -0.0000108 1.5708006"/>
+            <geometry>
+                <box size="0.032 0.042 0.023"/>
             </geometry>
             <material name="white"/>
@@ -486,14 +472,14 @@
         </visual>
         <visual>
-            <origin xyz="0.006 0.0 -0.054"/>
-            <geometry>
-                <box size="0.032 0.042 0.0225" rpy="0.654047 0.654046 0.380062 2.415205"/>
-            </geometry>
-            <material name="white"/>
-        </visual>
-        <visual>
-            <origin xyz="0.003 0 -0.037"/>
-            <geometry>
-                <box size="0.0465 0.036 0.02" rpy="-0.697151 -0.697152 -0.167211 -2.810252"/>
+            <origin xyz="0.006 0.0 -0.054" rpy="2.0887992 -0.0000101 1.5708007"/>
+            <geometry>
+                <box size="0.032 0.042 0.0225"/>
+            </geometry>
+            <material name="white"/>
+        </visual>
+        <visual>
+            <origin xyz="0.003 0 -0.037" rpy="2.6707995 -0.0000107 1.5708003"/>
+            <geometry>
+                <box size="0.0465 0.036 0.02"/>
             </geometry>
             <material name="white"/>
@@ -509,7 +495,7 @@
     <link name="right_knee_link">
         <visual>
-            <origin xyz="0.00425 0 -0.008"/>
-            <geometry>
-                <box size="0.0465 0.036 0.02"  rpy=" 0.454459 0.454452 0.76612 1.834125"/>
+            <origin xyz="0.00425 0 -0.008" rpy="1.0707999 -0.000011 1.5707994"/>
+            <geometry>
+                <box size="0.0465 0.036 0.02"/>
             </geometry>
             <material name="white"/>
@@ -523,7 +509,7 @@
         </visual>
         <visual>
-            <origin xyz="0.004 0.0 -0.054"/>
-            <geometry>
-                <box size="0.032 0.042 0.023"  rpy="-0.63513 -0.635128 -0.43957 -2.313314"/>
+            <origin xyz="0.004 0.0 -0.054" rpy="1.9307994 -0.0000108 1.5708006"/>
+            <geometry>
+                <box size="0.032 0.042 0.023"/>
             </geometry>
             <material name="white"/>
