Commit message: starting to implement controller now!

File: ros/src/uvc_robot_description/description/robot_core.xacro (robot description, xacro)
@@ -659,18 +659,18 @@
     <link name="left_foot_link">
         <visual>
-            <origin xyz="0 0.0265 -0.01825"/>
-            <geometry>
-                <box size="0.108 0.071 0.0165"/>
-            </geometry>
-            <material name="white"/>
-        </visual>
-        <collision>
-            <origin xyz="0 0.0265 -0.01825"/>
-            <geometry>
-                <box size="0.108 0.071 0.0165"/>
-            </geometry>
-        </collision>
-        <xacro:inertial_box mass="0.5" x="0.108" y="0.071" z="0.0165">
-            <origin xyz="0 0.0265 -0.01825"/>
+            <origin xyz="0 0.01125 -0.01825"/>
+            <geometry>
+                <box size="0.04 0.0425 0.0165"/>
+            </geometry>
+            <material name="white"/>
+        </visual>
+        <collision>
+           <origin xyz="0 0.01125 -0.01825"/>
+            <geometry>
+                <box size="0.04 0.0425 0.0165"/>
+            </geometry>
+        </collision>
+        <xacro:inertial_box mass="0.5" x="0.04" y="0.0425" z="0.0165">
+            <origin xyz="0 0.01125 -0.01825"/>
         </xacro:inertial_box>
     </link>
@@ -894,18 +894,18 @@
     <link name="right_foot_link">
         <visual>
-            <origin xyz="0 -0.0265 -0.01825"/>
-            <geometry>
-                <box size="0.108 0.071 0.0165"/>
-            </geometry>
-            <material name="white"/>
-        </visual>
-        <collision>
-            <origin xyz="0 -0.0265 -0.01825"/>
-            <geometry>
-                <box size="0.108 0.071 0.0165"/>
-            </geometry>
-        </collision>
-        <xacro:inertial_box mass="0.5" x="0.108" y="0.071" z="0.0165">
-            <origin xyz="0 -0.0265 -0.01825"/>
+            <origin xyz="0 -0.01125 -0.01825"/>
+            <geometry>
+                <box size="0.04 0.0425 0.0165"/>
+            </geometry>
+            <material name="white"/>
+        </visual>
+        <collision>
+            <origin xyz="0 -0.01125 -0.01825"/>
+            <geometry>
+                <box size="0.04 0.0425 0.0165"/>
+            </geometry>
+        </collision>
+        <xacro:inertial_box mass="0.5" x="0.04" y="0.0425" z="0.0165">
+            <origin xyz="0 -0.01125 -0.01825"/>
         </xacro:inertial_box>
     </link>

File: ros/src/uvc_robot_description/description/ros2_control.xacro (robot description, xacro)
@@ -6,221 +6,111 @@
             </hardware>
             <joint name="waist_joint">
-                <command_interface name="effort">
-                    <param name="min">-10</param>
-                    <param name="max">10</param>
-                </command_interface>
                 <command_interface name="position"/>
                 <state_interface name="effort"/>
-                <state_interface name="velocity"/>
                 <state_interface name="position"/>
             </joint>
             <joint name="head_joint">
-                <command_interface name="effort">
-                    <param name="min">-10</param>
-                    <param name="max">10</param>
-                </command_interface>
                 <command_interface name="position"/>
                 <state_interface name="effort"/>
-                <state_interface name="velocity"/>
                 <state_interface name="position"/>
             </joint>
             <joint name="left_shoulder_joint">
-                <command_interface name="effort">
-                    <param name="min">-10</param>
-                    <param name="max">10</param>
-                </command_interface>
                 <command_interface name="position"/>
                 <state_interface name="effort"/>
-                <state_interface name="velocity"/>
                 <state_interface name="position"/>
             </joint>
             <joint name="left_arm_joint">
-                <command_interface name="effort">
-                    <param name="min">-10</param>
-                    <param name="max">10</param>
-                </command_interface>
                 <command_interface name="position"/>
                 <state_interface name="effort"/>
-                <state_interface name="velocity"/>
                 <state_interface name="position"/>
             </joint>
             <joint name="left_elbow_joint">
-                <command_interface name="effort">
-                    <param name="min">-10</param>
-                    <param name="max">10</param>
-                </command_interface>
                 <command_interface name="position"/>
                 <state_interface name="effort"/>
-                <state_interface name="velocity"/>
                 <state_interface name="position"/>
             </joint>
             <joint name="left_forearm_joint">
-                <command_interface name="effort">
-                    <param name="min">-10</param>
-                    <param name="max">10</param>
-                </command_interface>
                 <command_interface name="position"/>
                 <state_interface name="effort"/>
-                <state_interface name="velocity"/>
                 <state_interface name="position"/>
             </joint>
             <joint name="right_shoulder_joint">
-                <command_interface name="effort">
-                    <param name="min">-10</param>
-                    <param name="max">10</param>
-                </command_interface>
                 <command_interface name="position"/>
                 <state_interface name="effort"/>
-                <state_interface name="velocity"/>
                 <state_interface name="position"/>
             </joint>
             <joint name="right_arm_joint">
-                <command_interface name="effort">
-                    <param name="min">-10</param>
-                    <param name="max">10</param>
-                </command_interface>
                 <command_interface name="position"/>
                 <state_interface name="effort"/>
-                <state_interface name="velocity"/>
                 <state_interface name="position"/>
             </joint>
             <joint name="right_elbow_joint">
-                <command_interface name="effort">
-                    <param name="min">-10</param>
-                    <param name="max">10</param>
-                </command_interface>
                 <command_interface name="position"/>
                 <state_interface name="effort"/>
-                <state_interface name="velocity"/>
                 <state_interface name="position"/>
             </joint>
             <joint name="right_forearm_joint">
-                <command_interface name="effort">
-                    <param name="min">-10</param>
-                    <param name="max">10</param>
-                </command_interface>
                 <command_interface name="position"/>
                 <state_interface name="effort"/>
-                <state_interface name="velocity"/>
                 <state_interface name="position"/>
             </joint>
             <joint name="left_hip1_joint">
-                <command_interface name="effort">
-                    <param name="min">-10</param>
-                    <param name="max">10</param>
-                </command_interface>
                 <command_interface name="position"/>
                 <state_interface name="effort"/>
-                <state_interface name="velocity"/>
                 <state_interface name="position"/>
             </joint>
             <joint name="left_hip2_joint">
-                <command_interface name="effort">
-                    <param name="min">-10</param>
-                    <param name="max">10</param>
-                </command_interface>
                 <command_interface name="position"/>
                 <state_interface name="effort"/>
-                <state_interface name="velocity"/>
                 <state_interface name="position"/>
             </joint>
             <joint name="left_leg_joint">
-                <command_interface name="effort">
-                    <param name="min">-10</param>
-                    <param name="max">10</param>
-                </command_interface>
                 <command_interface name="position"/>
                 <state_interface name="effort"/>
-                <state_interface name="velocity"/>
                 <state_interface name="position"/>
             </joint>
             <joint name="left_knee_joint">
-                <command_interface name="effort">
-                    <param name="min">-10</param>
-                    <param name="max">10</param>
-                </command_interface>
                 <command_interface name="position"/>
                 <state_interface name="effort"/>
-                <state_interface name="velocity"/>
                 <state_interface name="position"/>
             </joint>
             <joint name="left_ankle_joint">
-                <command_interface name="effort">
-                    <param name="min">-10</param>
-                    <param name="max">10</param>
-                </command_interface>
                 <command_interface name="position"/>
                 <state_interface name="effort"/>
-                <state_interface name="velocity"/>
                 <state_interface name="position"/>
             </joint>
             <joint name="left_foot_joint">
-                <command_interface name="effort">
-                    <param name="min">-10</param>
-                    <param name="max">10</param>
-                </command_interface>
                 <command_interface name="position"/>
                 <state_interface name="effort"/>
-                <state_interface name="velocity"/>
                 <state_interface name="position"/>
             </joint>
             <joint name="right_hip1_joint">
-                <command_interface name="effort">
-                    <param name="min">-10</param>
-                    <param name="max">10</param>
-                </command_interface>
                 <command_interface name="position"/>
                 <state_interface name="effort"/>
-                <state_interface name="velocity"/>
                 <state_interface name="position"/>
             </joint>
             <joint name="right_hip2_joint">
-                <command_interface name="effort">
-                    <param name="min">-10</param>
-                    <param name="max">10</param>
-                </command_interface>
                 <command_interface name="position"/>
                 <state_interface name="effort"/>
-                <state_interface name="velocity"/>
                 <state_interface name="position"/>
             </joint>
             <joint name="right_leg_joint">
-                <command_interface name="effort">
-                    <param name="min">-10</param>
-                    <param name="max">10</param>
-                </command_interface>
                 <command_interface name="position"/>
                 <state_interface name="effort"/>
-                <state_interface name="velocity"/>
                 <state_interface name="position"/>
             </joint>
             <joint name="right_knee_joint">
-                <command_interface name="effort">
-                    <param name="min">-10</param>
-                    <param name="max">10</param>
-                </command_interface>
                 <command_interface name="position"/>
                 <state_interface name="effort"/>
-                <state_interface name="velocity"/>
                 <state_interface name="position"/>
             </joint>
             <joint name="right_ankle_joint">
-                <command_interface name="effort">
-                    <param name="min">-10</param>
-                    <param name="max">10</param>
-                </command_interface>
                 <command_interface name="position"/>
                 <state_interface name="effort"/>
-                <state_interface name="velocity"/>
                 <state_interface name="position"/>
             </joint>
             <joint name="right_foot_joint">
-                <command_interface name="effort">
-                    <param name="min">-10</param>
-                    <param name="max">10</param>
-                </command_interface>
                 <command_interface name="position"/>
                 <state_interface name="effort"/>
-                <state_interface name="velocity"/>
                 <state_interface name="position"/>
             </joint>
